File: hardware/kicad/ecu25-main/analog.kicad_sch (KiCad schematic)
At the start: 41 parts, among them J13 Screw_Terminal_DPLUS, J3 Screw_Terminal_SENDERS, Q3 BC857, Q4 BC857, Q5 BC857, U3 LM358, U4 LM358

Commit message: Assign footprints to all 299 components in schematic generator
- By-ref exceptions + per-symbol defaults + value rules (wattage/voltage classes)
- Field connectors: MKDS-3 for battery/AC/CT/relay terminals, MKDS-1,5 for signal
- Q1 reverse-protection FET: Q_PMOS_GSD -> Q_PMOS_GDS + TO-252-2 (DPAK pad
  numbering 1=G 2=D 3=S; GSD variant would swap D/S in the netlist), part
  SQD50P06-15L
- Verified: all footprint files exist in KiCad 7 libs, all symbol pin numbers
  present in footprint pads, netlist sweep still clean
Parts:
- C20, C21, C22, C60, C63, C64, C85, C86: footprint (none) -> Capacitor_SMD:C_0603_1608Metric
- D20, D21, D22, D81, D82, Q3, Q4, Q5: footprint (none) -> Package_TO_SOT_SMD:SOT-23
- J13: footprint (none) -> TerminalBlock_Phoenix:TerminalBlock_Phoenix_MKDS-1,5-2-5.08_1x02_P5.08mm_Horizontal
- J3: footprint (none) -> TerminalBlock_Phoenix:TerminalBlock_Phoenix_MKDS-1,5-4-5.08_1x04_P5.08mm_Horizontal
- R18, R185, R186, R187, R19, R20, R21, R22, R23, R24, R25, R26, R27, R28, R29, R70, R71, R85, R86, R87: footprint (none) -> Resistor_SMD:R_0603_1608Metric
- R88: footprint (none) -> Resistor_THT:R_Axial_Power_L25.0mm_W9.0mm_P30.48mm
- U3, U4: footprint (none) -> Package_SO:SOIC-8_3.9x4.9mm_P1.27mm
