File: hardware/kicad/ecu25-main/analog.kicad_sch (KiCad schematic)
At the start: 41 parts, among them J13 Screw_Terminal_DPLUS, J3 Screw_Terminal_SENDERS, Q3 BC857, Q4 BC857, Q5 BC857, U3 LM358, U4 LM358

Commit message: Convert hardware to 12 V system; pilot-duty output stage
The target set is a Kirloskar KG4-25WS1 (engine 3R550ETA 4G1, CPCB IV+):
12 V electrical system, 75 Ah battery, 3-cylinder CRDi with EGR + DOC.
The board was designed 24 V throughout, which was wrong.

Power:
- Rails renamed +24V/+24V_SW -> +12V/+12V_SW
- Buck UVLO 8.0 V -> 6.5 V (R3 30.1k), RON 100k -> 49.9k to hold ~300 kHz
  from a 12 V input
- New D3 blocking Schottky + C9 2200uF hold-up on the buck input. UVLO now
  senses the hold-up node, not the battery: sensing the battery would trip EN
  the moment the harness sagged during crank and switch the buck off while C9
  still held charge. Sized for >50 ms down to 6.5 V with the backlight shed
- Input protection rescaled for 12 V: D1 SMCJ33CA -> SMCJ16CA (clamps ~26 V
  not 53 V), D80 -> SMBJ16CA, D2 gate zener 15 V -> 12 V, C1 63 V -> 35 V

Outputs — the board no longer sources any field current:
- J8 becomes a 6-pole body with 5 poles wired: pin 1 OUT_COM is the common
  contact supply, fed by the INSTALLER from a fused source. Relay contact COMs
  come from it, not from the board rail
- +12V_SW now feeds only the six relay coils (200 mA) and D+ (100 mA)
- START marked pilot-only: a 12 V starter solenoid pulls 20-40 A and glow
  plugs 28-60 A, against 8 A DC contacts
- K5/K6 HORN/PREHEAT -> configurable AUX1/AUX2; on a CRDi engine the ECU owns
  the cold-start aid, so a fixed preheat channel would often go unused
- Relay coils G5LE-1-DC24 -> DC12 (360 ohm / 33 mA)

Analog rescaled for 12 V:
- DIN dividers 10k/3.3k -> 5.6k/1.8k, restoring 1.6 mA contact wetting
  (10k/3.3k gives only 0.9 mA at 12 V), debounce cap 470 nF -> 1 uF
- Battery and D+ sense 100k/6.8k -> 100k/22k, so 16 V uses most of the ADC span
- D+ excitation 220R 5W -> 120R 3W for the same 100 mA at 12 V

Verified: netlist sweep clean, no courtyard overlaps, nothing outside the
outline, DRC reports no errors (unrouted ratsnest and silk warnings aside).
Docs and firmware follow in the next com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
Parts:
- R186, R86: value 6.8k 1% -> 22k 1%
- R88: value 220R 5W -> 120R 3W; footprint Resistor_THT:R_Axial_Power_L25.0mm_W9.0mm_P30.48mm -> Resistor_THT:R_Axial_Power_L20.0mm_W6.4mm_P25.40mm
Connections:
- net +24V renamed +12V
- net +24V_SW renamed +12V_SW
Other:
- note added: "LM358 V+ = +12V: input CM range must stay >=1.5V below V+; 4.5V ref OK. Current source from +5V rail."
- note removed: "LM358 V+ = +24V: input CM range must stay >=1.5V below V+; 4.5V ref OK. Current source from +5V rail."
