File: hardware/kicad/ecu25-main/digital.kicad_sch (KiCad schematic)
At the start: 71 parts, among them J2 Screw_Terminal_DIN, J4 Screw_Terminal_MPU, U5 LM2903

Commit message: Fix SME review findings: 3 critical, 6 major schematic faults
Critical:
- RON pin no longer shorted to GND (R4 moved off C3's column)
- LM2903 MPU comparator +/- inputs unmerged (separate route columns)
- Supercap charge diode D70 un-reversed (anode to +3V3)

Major:
- Buck UVLO divider restored (stray EN stub ended on C3 column = EN
  tied to +24V; stub removed)
- RS485 fail-safe bias polarity corrected (pull-up A, pull-down B)
- U8 spare op-amp unit placed and tied off (was floating on VREF die)
- Heartbeat LED DS1 un-reversed
- VREF_MID buffer dual feedback added (R93 DC path + C93 AC path)
- D80 value SMBJ33A -> SMBJ33CA (bidirectional, matches symbol)

Added netlist-level sweep check (shorted 2-pin devices, rail
membership) since the geometric tracer is blind to shorts closed
through power symbols across wire islands. Sweep: CLEAN, 0 issues.
Connections:
- net at D30.3 (K), R30.2, R31.2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: no longer R33.2, R34.1, U5.2 (-)
- new net: R33.2, R34.1, U5.2 (-)

Commit message: Assign footprints to all 299 components in schematic generator
- By-ref exceptions + per-symbol defaults + value rules (wattage/voltage classes)
- Field connectors: MKDS-3 for battery/AC/CT/relay terminals, MKDS-1,5 for signal
- Q1 reverse-protection FET: Q_PMOS_GSD -> Q_PMOS_GDS + TO-252-2 (DPAK pad
  numbering 1=G 2=D 3=S; GSD variant would swap D/S in the netlist), part
  SQD50P06-15L
- Verified: all footprint files exist in KiCad 7 libs, all symbol pin numbers
  present in footprint pads, netlist sweep still clean
Parts:
- C201, C202, C203, C204, C205, C206, C207, C208, C31: footprint (none) -> Capacitor_SMD:C_0603_1608Metric
- C30: footprint (none) -> Capacitor_SMD:C_0805_2012Metric
- D10, D11, D12, D13, D14, D15, D16, D17, D30: footprint (none) -> Package_TO_SOT_SMD:SOT-23
- J2: footprint (none) -> TerminalBlock_Phoenix:TerminalBlock_Phoenix_MKDS-1,5-10-5.08_1x10_P5.08mm_Horizontal
- J4: footprint (none) -> TerminalBlock_Phoenix:TerminalBlock_Phoenix_MKDS-1,5-2-5.08_1x02_P5.08mm_Horizontal
- JP10, JP11, JP4, JP5, JP6, JP7, JP8, JP9: footprint (none) -> Jumper:SolderJumper-2_P1.3mm_Open_RoundedPad1.0x1.5mm
- R201, R202, R203, R204, R205, R206, R207, R208, R231, R232, R233, R234, R235, R236, R237, R238: footprint (none) -> Resistor_SMD:R_1210_3225Metric
- R211, R212, R213, R214, R215, R216, R217, R218, R221, R222, R223, R224, R225, R226, R227, R228, R30, R31, R32, R33, R34, R35, R36, R37, R38: footprint (none) -> Resistor_SMD:R_0603_1608Metric
- U5: footprint (none) -> Package_SO:SOIC-8_3.9x4.9mm_P1.27mm
