File: hardware/kicad/ecu25-main/digital.kicad_sch (KiCad schematic)
At the start: 71 parts, among them J2 Screw_Terminal_DIN, J4 Screw_Terminal_MPU, U5 LM2903

Commit message: Convert hardware to 12 V system; pilot-duty output stage
The target set is a Kirloskar KG4-25WS1 (engine 3R550ETA 4G1, CPCB IV+):
12 V electrical system, 75 Ah battery, 3-cylinder CRDi with EGR + DOC.
The board was designed 24 V throughout, which was wrong.

Power:
- Rails renamed +24V/+24V_SW -> +12V/+12V_SW
- Buck UVLO 8.0 V -> 6.5 V (R3 30.1k), RON 100k -> 49.9k to hold ~300 kHz
  from a 12 V input
- New D3 blocking Schottky + C9 2200uF hold-up on the buck input. UVLO now
  senses the hold-up node, not the battery: sensing the battery would trip EN
  the moment the harness sagged during crank and switch the buck off while C9
  still held charge. Sized for >50 ms down to 6.5 V with the backlight shed
- Input protection rescaled for 12 V: D1 SMCJ33CA -> SMCJ16CA (clamps ~26 V
  not 53 V), D80 -> SMBJ16CA, D2 gate zener 15 V -> 12 V, C1 63 V -> 35 V

Outputs — the board no longer sources any field current:
- J8 becomes a 6-pole body with 5 poles wired: pin 1 OUT_COM is the common
  contact supply, fed by the INSTALLER from a fused source. Relay contact COMs
  come from it, not from the board rail
- +12V_SW now feeds only the six relay coils (200 mA) and D+ (100 mA)
- START marked pilot-only: a 12 V starter solenoid pulls 20-40 A and glow
  plugs 28-60 A, against 8 A DC contacts
- K5/K6 HORN/PREHEAT -> configurable AUX1/AUX2; on a CRDi engine the ECU owns
  the cold-start aid, so a fixed preheat channel would often go unused
- Relay coils G5LE-1-DC24 -> DC12 (360 ohm / 33 mA)

Analog rescaled for 12 V:
- DIN dividers 10k/3.3k -> 5.6k/1.8k, restoring 1.6 mA contact wetting
  (10k/3.3k gives only 0.9 mA at 12 V), debounce cap 470 nF -> 1 uF
- Battery and D+ sense 100k/6.8k -> 100k/22k, so 16 V uses most of the ADC span
- D+ excitation 220R 5W -> 120R 3W for the same 100 mA at 12 V

Verified: netlist sweep clean, no courtyard overlaps, nothing outside the
outline, DRC reports no errors (unrouted ratsnest and silk warnings aside).
Docs and firmware follow in the next com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
Parts:
- C201, C202, C203, C204, C205, C206, C207, C208: value 470nF -> 1uF 50V
- R201, R202, R203, R204, R205, R206, R207, R208, R231, R232, R233, R234, R235, R236, R237, R238: value 10k 0.5W -> 5.6k 0.5W
- R211, R212, R213, R214, R215, R216, R217, R218: value 3.3k -> 1.8k
Connections:
- net +24V renamed +12V
Other:
- note added: "J2: DIN1..DIN8 + 2x GND. Switch to +12V (default) or GND (fit JP per channel)."
- note removed: "J2: DIN1..DIN8 + 2x GND. Switch to +24V (default) or GND (fit JP per channel)."

Commit message: Fix SME review findings on the 12 V conversion
Two criticals, both of which would have reached a real installation:

- gcu_config.c still carried 24 V battery thresholds (22 V low / 30 V high).
  On a 12 V set batt_low was permanently true, so 60 s after every power-up
  the alarm latched and pinned the horn relay on for good — while batt_high
  at 30 V could never trip, leaving a runaway regulator undetected exactly
  where the new 16 V TVS starts conducting. Now 11.0 / 15.5 V, with a
  regression test that runs 90 s at 13.8 V and asserts silence
- docs/ecu-25-explained.md still told the installer to wire the starter
  solenoid straight to K2 at '16 A'. A G5LE-1 is 8 A DC and a 12 V starter
  solenoid pulls 20-40 A: the contacts weld, and a welded starter contact
  means the engine cranks and cannot be commanded to stop. Section rewritten
  around the dry-contact stage

Majors:
- gen_pcb.py netclass patterns still named +24V/+24V_SW, so the battery rail,
  the switched rail, the hold-up node and OUT_COM all fell through to a
  0.25 mm Default track — OUT_COM being the common return for every field
  contact. Fixed, and the generator now fails if any netclass pattern matches
  no net, which is what would have caught it
- DIN ground-side pull-up 5.6k -> 2.2k: at 5.6k an open contact sat at 1.66 V,
  inside the STM32's indeterminate band (V_IL 1.12 / V_IH 1.79)
- Buck RON 49.9k -> 41.2k. The LM5164's f_SW = V_OUT x 2500 / R_RON has no
  V_IN term — on-time varies inversely with V_IN precisely so frequency stays
  constant — so the rationale in two documents was wrong, and the original
  100k was never 300 kHz at any input voltage, it was 125 kHz
- modbus_rx guarded resp_max >= 5 but the FC06/FC16 echo paths write 8 bytes,
  running three bytes past the caller's buffer. Guard raised to 8
- Modbus no longer publishes a fabricated power factor: registers 19/20 now
  carry real_power_w and power_factor from gcu_inputs_t, which the AC layer
  fills. A constant 0.800 in a S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
Parts:
- R231, R232, R233, R234, R235, R236, R237, R238: value 5.6k 0.5W -> 2.2k 0.5W

Commit message: Fix SME verification findings; add COT ripple injection and the I/O map
An independent verification pass re-derived the 12 V conversion fixes against
the TI, Omron, Nexperia and ST datasheets instead of trusting the commit
message. The hold-up energy math, the RON/UVLO arithmetic, the modbus_rx
bounds, the AUX refactor and the dry-contact output stage all held. Eleven
majors did not.

Hardware:
- The buck had no ripple-injection network. The LM5164 is constant-on-time:
  it restarts the on-time when FB falls to the 1.2 V reference, so it needs
  >=20 mV of FB ripple IN PHASE with the inductor current. Two 22 uF ceramics
  give 2.7 mV, and that component is capacitive, i.e. out of phase — the
  required series ESR would be 0.287 ohm against the ~2 mohm they actually
  have. The part would have burst-switched: several on-times in close
  succession then a long off-time. Added the datasheet's Type-3 network
  (R7 100k, C10 4.7nF, C11 1nF C0G), which builds the ramp from SW and
  couples it into FB, leaving output ripple untouched. 21 mV at 12.6 V in,
  13 mV at 8 V, against a 12 mV floor
- DIN ground-side pull-up 2.2k -> 1k. 2.2k sat at 2.25 V at 12.6 V but fell
  to 1.59 V during an 8.5 V crank sag — back inside the STM32's indeterminate
  band. The value has to be set by the worst case: V_bat x 1.8/(R+7.4) needs
  R <= 670 ohm to clear V_IH 1.785 V at 8.0 V
- The hold-up node was still the autogenerated Net-(D3-K), so the netclass
  rule and the DRU keyed off a reference designator. Now labelled +12V_HLD
- C9 25 V -> 35 V never reached the orderable BOM: gen_bom.py still said
  "2200 uF 25 V radial" for a node the design puts at 25.6 V
- OUT_COM moved to the Battery class and given a stated ceiling: 4 A total,
  2 A per output, installer fuse 4 A. Four 8 A contacts on a trunk sized for
  4 A needed writing down; it was implied by the netclass and nowhere else
- gen_pcb.py netclass assertion rewritten. It was blind to exactly the
  suffix patterns it was written to pr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
Parts:
- R231, R232, R233, R234, R235, R236, R237, R238: value 2.2k 0.5W -> 1k 0.5W
Other:
- note added: "8x 12V digital inputs (divider + clamp, fw debounce); MPU pickup -> LM2903 comparator with +/-80mV hysteresis."
- note removed: "8x 24V digital inputs (divider + clamp, fw debounce); MPU pickup -> LM2903 comparator with +/-80mV hysteresis."
