File: hardware/kicad/ecu25-main/display.kicad_sch (KiCad schematic)
At the start: 1 part, among them J12 Ribbon 20-way

Commit message: Assign footprints to all 299 components in schematic generator
- By-ref exceptions + per-symbol defaults + value rules (wattage/voltage classes)
- Field connectors: MKDS-3 for battery/AC/CT/relay terminals, MKDS-1,5 for signal
- Q1 reverse-protection FET: Q_PMOS_GSD -> Q_PMOS_GDS + TO-252-2 (DPAK pad
  numbering 1=G 2=D 3=S; GSD variant would swap D/S in the netlist), part
  SQD50P06-15L
- Verified: all footprint files exist in KiCad 7 libs, all symbol pin numbers
  present in footprint pads, netlist sweep still clean
Parts:
- J12: footprint (none) -> Connector_IDC:IDC-Header_2x10-1MP_P2.54mm_Latch_Vertical
Changed lines of the file:
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@@
       (effects (font (size 1.27 1.27)) (justify left))
     )
-    (property "Footprint" "" (id 2) (at 119.38 90.17 0)
+    (property "Footprint" "Connector_IDC:IDC-Header_2x10-1MP_P2.54mm_Latch_Vertical" (id 2) (at 119.38 90.17 0)
       (effects (font (size 1.27 1.27)) hide)
     )
@@
     (instances
       (project "ecu25-main"
-        (path "/b289af85-c758-46d8-b7a5-0acd18d58c59/bdb12965-9206-4473-8c5b-2e518bda1e5e"
+        (path "/9fef0f12-125a-4195-98b7-20c6b2c3be48/87439dc0-73ba-4765-8173-0f57b60e0b84"
           (reference "J12") (unit 1)
         )
@@
     (instances
       (project "ecu25-main"
-        (path "/b289af85-c758-46d8-b7a5-0acd18d58c59/bdb12965-9206-4473-8c5b-2e518bda1e5e"
+        (path "/9fef0f12-125a-4195-98b7-20c6b2c3be48/87439dc0-73ba-4765-8173-0f57b60e0b84"
           (reference "#PWR226") (unit 1)
         )
@@
     (instances
       (project "ecu25-main"
-        (path "/b289af85-c758-46d8-b7a5-0acd18d58c59/bdb12965-9206-4473-8c5b-2e518bda1e5e"
+        (path "/9fef0f12-125a-4195-98b7-20c6b2c3be48/87439dc0-73ba-4765-8173-0f57b60e0b84"
           (reference "#PWR227") (unit 1)
         )
@@
     (instances
       (project "ecu25-main"
-        (path "/b289af85-c758-46d8-b7a5-0acd18d58c59/bdb12965-9206-4473-8c5b-2e518bda1e5e"
+        (path "/9fef0f12-125a-4195-98b7-20c6b2c3be48/87439dc0-73ba-4765-8173-0f57b60e0b84"
           (reference "#PWR228") (unit 1)
         )
@@
     (instances
       (project "ecu25-main"
-        (path "/b289af85-c758-46d8-b7a5-0acd18d58c59/bdb12965-9206-4473-8c5b-2e518bda1e5e"
+        (path "/9fef0f12-125a-4195-98b7-20c6b2c3be48/87439dc0-73ba-4765-8173-0f57b60e0b84"
           (reference "#PWR229") (unit 1)
         )
@@
     (instances
       (project "ecu25-main"
-        (path "/b289af85-c758-46d8-b7a5-0acd18d58c59/bdb12965-9206-4473-8c5b-2e518bda1e5e"
+        (path "/9fef0f12-125a-4195-98b7-20c6b2c3be48/87439dc0-73ba-4765-8173-0f57b60e0b84"
           (reference "#PWR230") (unit 1)
         )
@@
     (instances
       (project "ecu25-main"
-        (path "/b289af85-c758-46d8-b7a5-0acd18d58c59/bdb12965-9206-4473-8c5b-2e518bda1e5e"
+        (path "/9fef0f12-125a-4195-98b7-20c6b2c3be48/87439dc0-73ba-4765-8173-0f57b60e0b84"
           (reference "#PWR231") (unit 1)
         )
@@
     (instances
       (project "ecu25-main"
-        (path "/b289af85-c758-46d8-b7a5-0acd18d58c59/bdb12965-9206-4473-8c5b-2e518bda1e5e"
+        (path "/9fef0f12-125a-4195-98b7-20c6b2c3be48/87439dc0-73ba-4765-8173-0f57b60e0b84"
           (reference "#PWR232") (unit 1)
         )
@@
     (instances
       (project "ecu25-main"
-        (path "/b289af85-c758-46d8-b7a5-0acd18d58c59/bdb12965-9206-4473-8c5b-2e518bda1e5e"
+        (path "/9fef0f12-125a-4195-98b7-20c6b2c3be48/87439dc0-73ba-4765-8173-0f57b60e0b84"
           (reference "#PWR233") (unit 1)
         )
@@
     (instances
       (project "ecu25-main"
-        (path "/b289af85-c758-46d8-b7a5-0acd18d58c59/bdb12965-9206-4473-8c5b-2e518bda1e5e"
+        (path "/9fef0f12-125a-4195-98b7-20c6b2c3be48/87439dc0-73ba-4765-8173-0f57b60e0b84"
           (reference "#PWR234") (unit 1)
         )
@@
     (instances
       (project "ecu25-main"
-        (path "/b289af85-c758-46d8-b7a5-0acd18d58c59/bdb12965-9206-4473-8c5b-2e518bda1e5e"
+        (path "/9fef0f12-125a-4195-98b7-20c6b2c3be48/87439dc0-73ba-4765-8173-0f57b60e0b84"
           (reference "#PWR235") (unit 1)
         )
@@
     (instances
       (project "ecu25-main"
-        (path "/b289af85-c758-46d8-b7a5-0acd18d58c59/bdb12965-9206-4473-8c5b-2e518bda1e5e"
+        (path "/9fef0f12-125a-4195-98b7-20c6b2c3be48/87439dc0-73ba-4765-8173-0f57b60e0b84"
           (reference "#PWR236") (unit 1)
         )
