File: hardware/kicad/ecu25-main/ecu25-main.kicad_pcb (KiCad board)
At the start: 2 copper layers, 200 x 150 mm, 304 parts, among them J1 Screw_Terminal_BATT, J10 Screw_Terminal_RS485, J11 TC2030 SWD, J12 Ribbon 20-way, J13 Screw_Terminal_DPLUS, J14 DEBUG_UART, J15 Screw_Terminal_CONTACTOR, J2 Screw_Terminal_DIN, J3 Screw_Terminal_SENDERS, J4 Screw_Terminal_MPU, J5 Screw_Terminal_GEN, J6 Screw_Terminal_MAINS, J7 Screw_Terminal_CT, J8 Screw_Terminal_RELAY_OUT, J9 Screw_Terminal_CAN, K1 G5LE-1 24V, K2 G5LE-1 24V, K3 G5LE-1 24V, K4 G5LE-1 24V, K5 G5LE-1 24V, K6 G5LE-1 24V, Q1 SQD50P06-15L, Q3 BC857, Q4 BC857, Q5 BC857, Q60 2N7002K 60V, Q61 2N7002K 60V, Q62 2N7002K 60V, Q63 2N7002K 60V, Q64 2N7002K 60V, Q65 2N7002K 60V, U1 LM5164DDA-Q1, U10 MCP6002, U11 M95M02-DR, U12 STM32F407VGT6, U2 TLV75533 (500mA), U3 LM358, U4 LM358, U5 LM2903, U6 TJA1051T/3, U7 THVD1450, U8 MCP6002, U9 MCP6002, Y1 8MHz, Y2 32.768kHz

Commit message: Convert hardware to 12 V system; pilot-duty output stage
The target set is a Kirloskar KG4-25WS1 (engine 3R550ETA 4G1, CPCB IV+):
12 V electrical system, 75 Ah battery, 3-cylinder CRDi with EGR + DOC.
The board was designed 24 V throughout, which was wrong.

Power:
- Rails renamed +24V/+24V_SW -> +12V/+12V_SW
- Buck UVLO 8.0 V -> 6.5 V (R3 30.1k), RON 100k -> 49.9k to hold ~300 kHz
  from a 12 V input
- New D3 blocking Schottky + C9 2200uF hold-up on the buck input. UVLO now
  senses the hold-up node, not the battery: sensing the battery would trip EN
  the moment the harness sagged during crank and switch the buck off while C9
  still held charge. Sized for >50 ms down to 6.5 V with the backlight shed
- Input protection rescaled for 12 V: D1 SMCJ33CA -> SMCJ16CA (clamps ~26 V
  not 53 V), D80 -> SMBJ16CA, D2 gate zener 15 V -> 12 V, C1 63 V -> 35 V

Outputs — the board no longer sources any field current:
- J8 becomes a 6-pole body with 5 poles wired: pin 1 OUT_COM is the common
  contact supply, fed by the INSTALLER from a fused source. Relay contact COMs
  come from it, not from the board rail
- +12V_SW now feeds only the six relay coils (200 mA) and D+ (100 mA)
- START marked pilot-only: a 12 V starter solenoid pulls 20-40 A and glow
  plugs 28-60 A, against 8 A DC contacts
- K5/K6 HORN/PREHEAT -> configurable AUX1/AUX2; on a CRDi engine the ECU owns
  the cold-start aid, so a fixed preheat channel would often go unused
- Relay coils G5LE-1-DC24 -> DC12 (360 ohm / 33 mA)

Analog rescaled for 12 V:
- DIN dividers 10k/3.3k -> 5.6k/1.8k, restoring 1.6 mA contact wetting
  (10k/3.3k gives only 0.9 mA at 12 V), debounce cap 470 nF -> 1 uF
- Battery and D+ sense 100k/6.8k -> 100k/22k, so 16 V uses most of the ADC span
- D+ excitation 220R 5W -> 120R 3W for the same 100 mA at 12 V

Verified: netlist sweep clean, no courtyard overlaps, nothing outside the
outline, DRC reports no errors (unrouted ratsnest and silk warnings aside).
Docs and firmware follow in the next com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
Parts:
- added C9: 2200uF 25V, CP_Radial_D12.5mm_P5.00mm, F.Cu at (60.0, 62.0)
- added D3: SS34, D_SMA, F.Cu at (64.5, 38.4)
- C1: value 100uF 63V -> 100uF 35V; footprint CP_Radial_D10.0mm_P5.00mm -> CP_Radial_D8.0mm_P3.50mm
- C2: value 100nF 100V -> 100nF 50V; footprint C_0805_2012Metric -> C_0603_1608Metric
- C201, C202, C203, C204, C205, C206, C207, C208: value 470nF -> 1uF 50V
- C3: value 2.2uF 100V -> 2.2uF 50V
- D1: value SMCJ33CA -> SMCJ16CA
- D2: value BZT52C15 -> BZT52C12
- D80: value SMBJ33CA -> SMBJ16CA
- J8: footprint TerminalBlock_Phoenix_MKDS-3-4-5.08_1x04_P5.08mm_Horizontal -> TerminalBlock_Phoenix_MKDS-3-6-5.08_1x06_P5.08mm_Horizontal
- K1, K2, K3, K4, K5, K6: value G5LE-1 24V -> G5LE-1 12V
- R186, R86: value 6.8k 1% -> 22k 1%
- R201, R202, R203, R204, R205, R206, R207, R208, R231, R232, R233, R234, R235, R236, R237, R238: value 10k 0.5W -> 5.6k 0.5W
- R211, R212, R213, R214, R215, R216, R217, R218: value 3.3k -> 1.8k
- R3: value 23.2k (UVLO 8V) -> 30.1k 1% (UVLO 6.5V)
- R4: value 100k (RON 300kHz) -> 49.9k 1% (RON 300kHz)
- R88: value 220R 5W -> 120R 3W; footprint R_Axial_Power_L25.0mm_W9.0mm_P30.48mm -> R_Axial_Power_L20.0mm_W6.4mm_P25.40mm
- moved R2 54.5 mm to (92.6, 43.1)
- moved R5 54.5 mm to (92.6, 45.8)
- moved R3 50.4 mm to (38.1, 45.8)
- moved R6 50.4 mm to (38.1, 48.5)
- moved C7 49.5 mm to (38.1, 43.1)
- moved R18 39.1 mm to (38.1, 77.0)
- moved R185 39.1 mm to (42.3, 77.0)
- moved R186 39.1 mm to (46.5, 77.0)
- moved R187 39.1 mm to (50.7, 77.0)
- moved Q3 38.3 mm to (43.6, 73.3)
- moved Q4 38.3 mm to (48.7, 73.3)
- moved D82 38.3 mm to (38.5, 73.3)
- moved R28 38.0 mm to (38.1, 79.7)
- moved R29 38.0 mm to (42.3, 79.7)
- moved R71 38.0 mm to (50.7, 79.7)
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Connections:
- net RLY_HORN renamed RLY_AUX1
- net RLY_PREHEAT renamed RLY_AUX2
- C1 pad 1: +24V -> +12V
- C2 pad 1: +24V -> +12V
- C3 pad 1: +24V -> Net-(D3-K)
- C63 pad 1: +24V -> +12V
- C64 pad 1: +24V -> +12V
- D60 pad 1: +24V_SW -> +12V_SW
- D61 pad 1: +24V_SW -> +12V_SW
- D62 pad 1: +24V_SW -> +12V_SW
- D63 pad 1: +24V_SW -> +12V_SW
- D64 pad 1: +24V_SW -> +12V_SW
- D65 pad 1: +24V_SW -> +12V_SW
- D80 pad 2: +24V_SW -> +12V_SW
- F2 pad 1: +24V -> +12V
- F2 pad 2: +24V_SW -> +12V_SW
- FB1 pad 2: +24V -> +12V
- J8 pad 1: /Relay drivers/FUEL_OUT -> /Relay drivers/OUT_COM
- J8 pad 2: /Relay drivers/START_OUT -> /Relay drivers/FUEL_OUT
- J8 pad 3: /Relay drivers/HORN_OUT -> /Relay drivers/START_OUT
- J8 pad 4: /Relay drivers/PREHEAT_OUT -> /Relay drivers/AUX1_OUT
- K1 pad 1: +24V_SW -> /Relay drivers/OUT_COM
- K1 pad 5: +24V_SW -> +12V_SW
- K2 pad 1: +24V_SW -> /Relay drivers/OUT_COM
- K2 pad 5: +24V_SW -> +12V_SW
- K3 pad 5: +24V_SW -> +12V_SW
- K4 pad 5: +24V_SW -> +12V_SW
- K5 pad 1: +24V_SW -> /Relay drivers/OUT_COM
- K5 pad 3: /Relay drivers/HORN_OUT -> /Relay drivers/AUX1_OUT
- K5 pad 5: +24V_SW -> +12V_SW
- K6 pad 1: +24V_SW -> /Relay drivers/OUT_COM
- K6 pad 3: /Relay drivers/PREHEAT_OUT -> /Relay drivers/AUX2_OUT
- K6 pad 5: +24V_SW -> +12V_SW
- R2 pad 1: +24V -> Net-(D3-K)
- R231 pad 1: +24V -> +12V
- R232 pad 1: +24V -> +12V
- R233 pad 1: +24V -> +12V
- R234 pad 1: +24V -> +12V
- R235 pad 1: +24V -> +12V
- R236 pad 1: +24V -> +12V
- R237 pad 1: +24V -> +12V
- R238 pad 1: +24V -> +12V
- R85 pad 1: +24V -> +12V
- R88 pad 1: +24V_SW -> +12V_SW
- U1 pad 2: +24V -> Net-(D3-K)
- U3 pad 8: +24V -> +12V
- U4 pad 8: +24V -> +12V

Commit message: Fix SME review findings on the 12 V conversion
Two criticals, both of which would have reached a real installation:

- gcu_config.c still carried 24 V battery thresholds (22 V low / 30 V high).
  On a 12 V set batt_low was permanently true, so 60 s after every power-up
  the alarm latched and pinned the horn relay on for good — while batt_high
  at 30 V could never trip, leaving a runaway regulator undetected exactly
  where the new 16 V TVS starts conducting. Now 11.0 / 15.5 V, with a
  regression test that runs 90 s at 13.8 V and asserts silence
- docs/ecu-25-explained.md still told the installer to wire the starter
  solenoid straight to K2 at '16 A'. A G5LE-1 is 8 A DC and a 12 V starter
  solenoid pulls 20-40 A: the contacts weld, and a welded starter contact
  means the engine cranks and cannot be commanded to stop. Section rewritten
  around the dry-contact stage

Majors:
- gen_pcb.py netclass patterns still named +24V/+24V_SW, so the battery rail,
  the switched rail, the hold-up node and OUT_COM all fell through to a
  0.25 mm Default track — OUT_COM being the common return for every field
  contact. Fixed, and the generator now fails if any netclass pattern matches
  no net, which is what would have caught it
- DIN ground-side pull-up 5.6k -> 2.2k: at 5.6k an open contact sat at 1.66 V,
  inside the STM32's indeterminate band (V_IL 1.12 / V_IH 1.79)
- Buck RON 49.9k -> 41.2k. The LM5164's f_SW = V_OUT x 2500 / R_RON has no
  V_IN term — on-time varies inversely with V_IN precisely so frequency stays
  constant — so the rationale in two documents was wrong, and the original
  100k was never 300 kHz at any input voltage, it was 125 kHz
- modbus_rx guarded resp_max >= 5 but the FC06/FC16 echo paths write 8 bytes,
  running three bytes past the caller's buffer. Guard raised to 8
- Modbus no longer publishes a fabricated power factor: registers 19/20 now
  carry real_power_w and power_factor from gcu_inputs_t, which the AC layer
  fills. A constant 0.800 in a S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
Parts:
- C2: value 100nF 50V -> 100nF
- C9: value 2200uF 25V -> 2200uF 35V
- F1: value 5A blade -> 3A blade
- R231, R232, R233, R234, R235, R236, R237, R238: value 5.6k 0.5W -> 2.2k 0.5W
- R4: value 49.9k 1% (RON 300kHz) -> 41.2k 1% (RON 300kHz)
Connections:
- J8 pad 6: (no net) -> /Relay drivers/OUT_COM
